File: Progetto Lidar.kicad_sch (KiCad schematic)
At the start: 44 parts, among them J1 CONN_LASER, J10 Conn_01x08, J2 CONN_RICEVITORE, J3 Conn_02x18_Odd_Even, J4 Conn_01x10, J5 Conn_01x08, J6 Conn_01x08, J7 Conn_01x08, J8 Conn_SPI, J9 Conn_01x08

Commit message: Corretto collegamento TDC_START
Connections:
- net ARD_GPIO_D34 is gone; now on net TDC_START: IC_0.D34, J3.15 (Pin_15)
Changed lines of the file:
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@@
     (effects (font (size 1.27 1.27)) (justify right bottom))
+  )
+  (label "TDC_START" (at 81.28 82.55 0)
+    (effects (font (size 1.27 1.27)) (justify left bottom))
   )
   (label "ARD_GPIO_D37" (at 82.55 240.03 180)
@@
     (effects (font (size 1.27 1.27)) (justify left bottom))
   )
-  (label "ARD_GPIO_D34" (at 41.91 237.49 0)
-    (effects (font (size 1.27 1.27)) (justify left bottom))
-  )
-  (label "ARD_GPIO_D34" (at 81.28 82.55 0)
-    (effects (font (size 1.27 1.27)) (justify left bottom))
-  )
   (label "ARD_GPIO_50" (at 81.28 41.91 0)
     (effects (font (size 1.27 1.27)) (justify left bottom))
@@
     (effects (font (size 1.27 1.27)) (justify left bottom))
   )
+  (label "TDC_START" (at 41.91 237.49 0)
+    (effects (font (size 1.27 1.27)) (justify left bottom))
+  )

Commit message: Corretto connessione TDC ENABLE
Connections:
- net SPI_CS: no longer IC_1.1 (ENABLE)
- net ARD_GPIO_D38 renamed TDC_EN
- net TDC_EN: now also IC_1.1 (ENABLE)
Changed lines of the file:
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@@
+    (effects (font (size 1.27 1.27)) (justify left bottom))
+  )
+  (label "TDC_EN" (at 41.91 242.57 0)
     (effects (font (size 1.27 1.27)) (justify left bottom))
   )
@@
     (effects (font (size 1.27 1.27)) (justify left bottom))
   )
+  (label "TDC_EN" (at 81.28 72.39 0)
+    (effects (font (size 1.27 1.27)) (justify left bottom))
+  )
   (label "ARD_GPIO_47" (at 81.28 49.53 0)
     (effects (font (size 1.27 1.27)) (justify left bottom))
@@
     (effects (font (size 1.27 1.27)) (justify left bottom))
   )
-  (label "SPI_CS" (at 298.45 35.56 0)
+  (label "TDC_EN" (at 298.45 35.56 0)
     (effects (font (size 1.27 1.27)) (justify left bottom))
   )
@@
     (effects (font (size 1.27 1.27)) (justify left bottom))
   )
-  (label "ARD_GPIO_D38" (at 81.28 72.39 0)
-    (effects (font (size 1.27 1.27)) (justify left bottom))
-  )
   (label "3V3_ARDUINO" (at 343.789 218.186 0)
     (effects (font (size 1.27 1.27)) (justify left bottom))
@@
     (effects (font (size 1.27 1.27)) (justify left bottom))
   )
-  (label "ARD_GPIO_D38" (at 41.91 242.57 0)
-    (effects (font (size 1.27 1.27)) (justify left bottom))
-  )
